File: LSwarm Drone PCB/esp32-c3.kicad_sch (KiCad schematic)
At the start: 6 parts, among them U5 ESP32-C3

Commit message: sync
Parts:
- added C28, C29: 12pF, symbol Device:C
- added C30, C31, C32, C33, C34, C36, C37: 100nF, symbol Device:C
- added C35: 10nF, symbol Device:C
- added L3: L, symbol Device:L
- added L4: 2nH, symbol Device:L
- added R10, R9: 22, symbol Device:R
- added R11, R12, R13: 10k, symbol Device:R
- added S1, S4: SKRPACE010, SKRPACE010:SW_SKRPACE010, symbol SKRPACE010:SKRPACE010
- added Y2: 40MHz, symbol Device:Crystal_GND24
Connections:
- net ESP32_GPIO_7 is gone; now on net RP2350_SPIO_MOSI: U5.13 (MTDO)
- net +3.3V: now also U5.17 (VDD3P3_CPU), C33.1, C34.1, C35.1, C36.1, C37.1, L4.2, R11.1, R12.1, R13.1
- net ESP32_40M_X0: now also U5.30 (XTAL_P), L3.1; no longer U5.29 (XTAL_N)
- net ESP32_40M_X1: now also U5.29 (XTAL_N), C28.1, Y2.3; no longer U5.30 (XTAL_P)
- net ESP32_CHIP_EN: now also C30.1, R12.2, S1.1
- net ESP32_GPIO_18: now also R9.2
- net ESP32_GPIO_19: now also R10.2
- net ESP32_GPIO_8: now also R11.2
- net ESP32_GPIO_9: now also C31.1, R13.2, S4.1
- net ESP32_VDD_3P3: now also C32.1, L4.1; no longer U5.17 (VDD3P3_CPU)
- net GND: now also C28.2, C29.2, C30.2, C31.2, C32.2, C33.2, C34.2, C35.2, C36.2, C37.2, S1.4, S4.4, Y2.2 (G), Y2.4 (G)
- net ESP32_VDD_SPI: now reaches C27.1, U5.18 (VDD_SPI)
- net ESP32_GPIO_10 renamed RP2350_SPIO_SS
- net ESP32_GPIO_2 renamed RP2350_SPIO_MOSI
- net ESP32_GPIO_6 renamed RP2350_SPIO_SCK
- new net: C29.1, L3.2, Y2.1
- new net ESP32_USB_DN: R10.1
- new net ESP32_USB_DP: R9.1
- no-connect marks 6 -> 10
Other:
- note added: "Near VDD & VDDA Pins"
- note added: "Near VDD_3P3"
- moved on the sheet: C27

Commit message: sync
Parts:
- removed R10, R9: 22, symbol Device:R
Connections:
- net ESP32_CHIP_EN renamed RP2350_GPIO_14
- net ESP32_GPIO_4: no longer names the net of U5.9 (MTMS)
- net ESP32_GPIO_5: no longer names the net of U5.10 (MTDI)
- net ESP32_GPIO_9 renamed RP2350_GPIO_15
- net ESP32_UORXD renamed RP2350_GPIO_16
- net ESP32_UOTXD renamed RP2350_GPIO_17
- net RP2350_SPIO_MOSI: no longer names the net of U5.13 (MTDO)
- net RP2350_SPIO_MOSI: no longer U5.6 (GPIO2)
- net RP2350_SPIO_SCK: no longer names the net of U5.12 (MTCK)
- net RP2350_SPIO_SS renamed RP2350_GPIO_13
- new net RP2350_GPIO_12: U5.6 (GPIO2)
- no-connect marks 10 -> 14
Other:
- moved on the sheet: ANT1, C25, C26, C31, L2, R13, S4
