File: LSwarm Drone PCB/peripherals.kicad_sch (KiCad schematic)
At the start: 0 parts

Commit message: sync
Parts:
- added C1, C2, C4, C6, C7, C8, C9: 100nF, symbol Device:C
- added C3: 1uF, symbol Device:C
- added C5: 10uF, symbol Device:C
- added J1: JST / BT2.0 Connector, Connector_JST:JST_PH_S2B-PH-K_1x02_P2.00mm_Horizontal, symbol Connector:Conn_01x02_Socket
- added R1: 470, symbol Device:R
- added U1: LSM6DSR, LSM6DSR:LGA-14L, symbol LSM6DSR:LSM6DSR
- added U2: BMP581, BMP581:BMP581, symbol BMP581:BMP581
- added U3, U4, U5, U6: SK6812MINI-E, symbol SK6812MINI-E:SK6812MINI-E
- added U7: TPS61023DRLR, TPS61023DRLR:SOT563-ORI, symbol TPS61023DRLR:TPS61023DRLR
Connections:
- new net: C5.2, C6.1
- new net: C4.1, U1.P$5 (VDDIO)
- new net: C2.1, C3.2
- new net: U4.P$4 (DOUT), U5.P$3 (DIN)
- new net: U5.P$4 (DOUT), U6.P$3 (DIN)
- new net: R1.1, U3.P$3 (DIN)
- new net: U3.P$4 (DOUT), U4.P$3 (DIN)
- new net: U1.P$10 (UNCONNECTED), U1.P$11 (UNCONNECTED)
- new net +3.3V: C1.1, C3.1, C4.2, U1.P$8 (VDD), U2.1 (VDDIO), U2.10 (VDD)
- new net +5V: C6.2, C7.2, C8.2, C9.2, U3.P$2 (VDD), U4.P$2 (VDD), U5.P$2 (VDD), U6.P$2 (VDD)
- new net GND: C1.2, C2.2, C5.1, C7.1, C8.1, C9.1, U1.P$2 (SDX), U1.P$3 (SCX), U1.P$6 (GND), U1.P$7 (GND), U2.3 (GND), U2.8 (GND), U2.9 (GND), U3.P$1 (GND), U4.P$1 (GND), U5.P$1 (GND), U6.P$1 (GND)
- new net RP2350_GPIO_10: U1.P$12 (CS)
- new net RP2350_GPIO_11: U2.6 (CSB)
- new net RP2350_GPIO_25: R1.2
- new net RP2350_GPIO_4: U2.7 (INT)
- new net RP2350_GPIO_5: U1.P$4 (INT1)
- new net RP2350_GPIO_6: U1.P$9 (INT2)
- new net RP2350_GPIO_7: U1.P$13 (SCL), U2.2 (SCK/SCL)
- new net RP2350_GPIO_8: U1.P$14 (SDA), U2.4 (SDI/SDA)
- new net RP2350_GPIO_9: U1.P$1 (SDO), U2.5 (SDO/ADR)
- no-connect marks 0 -> 1
