File: LSwarm Drone PCB/LSwarm Drone PCB.kicad_sch (KiCad schematic)
At the start: 128 parts, among them J1 Conn_01x04_Pin, J2 USB_C_Receptacle_USB2.0_16P, J3 JST / BT2.0 Connector, J4 Conn_01x02_Pin, J5 Conn_01x02_Pin, J6 Conn_01x02_Pin, J7 Conn_01x02_Pin, Q1 AO3400A, Q2 AO3400A, Q3 AO3400A, Q4 AO3400A, Q5 AO3401A, U1 RP2350A, U10 LSM6DSR, U11 BMP581, U12 AP2112K-3.3, U13 TPS61023DRLR, U14 SN74LVC1T45DBVR, U15 SK6812MINI-E, U16 SK6812MINI-E, U17 SK6812MINI-E, U18 SK6812MINI-E, U19 SK6812MINI-E, U4 W25Q128JVS, U6 ESP32-C3, Y1 12MHz, Y3 40MHz

Commit message: imported components correctly into the pcb wiring design
Parts:
- removed BUZZER1: MLT-5020, easyeda2kicad:BUZ-SMD_L5.0-W5.5-P4.60, symbol MLT-5020:MLT-5020
- removed S1: MSK12C02, MSK12C02:SW_MSK12C02, symbol MSK12C02:MSK12C02
- removed U15, U16, U17, U18, U19: SK6812MINI-E, symbol SK6812MINI-E:SK6812MINI-E
- added BUZZER2: MLT-5020, easyeda2kicad:BUZ-SMD_L5.0-W5.5-P4.60, symbol easyeda2kicad:MLT-5020
- added LED1, LED2, LED3, LED4, LED5: SK6812MINI-E_C5149201, easyeda2kicad:LED-SMD_4P-L3.2-W2.8-LS5.9_SK6812MINI-E, symbol easyeda2kicad:SK6812MINI-E_C5149201
- added SW1: MSK12C02, easyeda2kicad:SW-TH_MSK12C02, symbol easyeda2kicad:MSK12C02
- C10, C11, C12, C13, C14, C16, C17, C18, C19, C20, C21, C22, C23, C24, C25, C3, C38, C39, C4, C40, C41, C44, C46, C47, C48, C49, C5, C50, C51, C52, C53, C54, C55, C56, C57, C58, C59, C6, C60, C61, C62, C64, C65, C66, C67, C68, C7, C71, C8, C9: footprint (none) -> Capacitor_SMD:C_0603_1608Metric
- C15, C42, C43, C45, C63, C71Ceramic1: footprint (none) -> Capacitor_SMD:C_0805_2012Metric
- C72: footprint (none) -> Capacitor_Tantalum_SMD:CP_EIA-3528-21_Kemet-B
- J1: footprint (none) -> Connector_PinHeader_2.54mm:PinHeader_1x04_P2.54mm_Vertical
- J2: footprint (none) -> Connector_USB:USB_C_Receptacle_HRO_TYPE-C-31-M-12
- J4, J5, J6, J7: footprint (none) -> Connector_PinHeader_2.54mm:PinHeader_1x02_P2.54mm_Vertical
- L1, L5: footprint (none) -> Inductor_SMD:L_1210_3225Metric
- L6: footprint (none) -> Inductor_SMD:L_0805_2012Metric
- L7, L8: footprint (none) -> Inductor_SMD:L_0402_1005Metric
- R1, R10, R11, R12, R13, R14, R15, R16, R17, R18, R19, R2, R20, R21, R22, R23, R24, R25, R26, R27, R28, R3, R4, R5, R6, R7, R8, R9: footprint (none) -> Resistor_SMD:R_0603_1608Metric
- Y1, Y3: footprint (none) -> Crystal:Crystal_SMD_3225-4Pin_3.2x2.5mm
Connections:
- net +3.3V: now also LED1.3 (VDD)
- net +5V: now also LED2.3 (VDD), LED3.3 (VDD), LED4.3 (VDD), LED5.3 (VDD)
- net GND: now also BUZZER2.2 (-), LED1.1 (GND), LED2.1 (GND), LED3.1 (GND), LED4.1 (GND), LED5.1 (GND), SW1.3
- net at R27.2: now also BUZZER2.1 (+)
- net at R9.1: now also LED2.2 (DIN)
- net at Q5.1 (G), R28.1: now also SW1.2
- net at R10.1: now also LED1.2 (DIN)
- new net: LED2.4 (DOUT), LED3.2 (DIN)
- new net: LED3.4 (DOUT), LED4.2 (DIN)
- new net: LED4.4 (DOUT), LED5.2 (DIN)

Commit message: sync
Parts:
- removed Q5: AO3401A, Package_TO_SOT_SMD:SOT-23, symbol Transistor_FET:AO3401A
- added Q7: AO3407A, easyeda2kicad:SOT-23-3_L2.9-W1.6-P1.90-LS2.8-BR, symbol easyeda2kicad:AO3407A
Connections:
- net BATT+: now also Q7.2 (S)
- net BATT_SW+: now also Q7.3 (D)
- net at R28.1, SW1.2: now also Q7.1 (G)
Changed lines of the file:
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@@
 	)
 	(junction
+		(at 280.67 100.33)
+		(diameter 0)
+		(color 0 0 0 0)
+	)
+	(junction
 		(at 74.93 210.82)
 		(diameter 0)
@@
 	)
 	(junction
+		(at 365.76 224.79)
+		(diameter 0)
+		(color 0 0 0 0)
+	)
+	(junction
 		(at 87.63 246.38)
 		(diameter 0)
@@
 	)
 	(junction
-		(at 365.76 224.79)
-		(diameter 0)
-		(color 0 0 0 0)
-	)
-	(junction
 		(at 247.65 184.15)
 		(diameter 0)
@@
 	)
 	(junction
-		(at 360.68 232.41)
-		(diameter 0)
-		(color 0 0 0 0)
-	)
-	(junction
 		(at 53.34 264.16)
 		(diameter 0)
@@
 	)
 	(junction
+		(at 360.68 232.41)
+		(diameter 0)
+		(color 0 0 0 0)
+	)
+	(junction
 		(at 254 146.05)
 		(diameter 0)
@@
 	(wire
 		(pts
-			(xy 283.21 100.33) (xy 283.21 110.49)
-		)
-		(stroke
-			(width 0)
-			(type default)
-		)
-	)
-	(wire
-		(pts
 			(xy 48.26 137.16) (xy 54.61 137.16)
 		)
@@
 	(wire
 		(pts
+			(xy 285.75 100.33) (xy 285.75 110.49)
+		)
+		(stroke
+			(width 0)
+			(type default)
+		)
+	)
+	(wire
+		(pts
 			(xy 77.47 184.15) (xy 85.09 184.15)
 		)
@@
 	(wire
 		(pts
+			(xy 276.86 100.33) (xy 280.67 100.33)
+		)
+		(stroke
+			(width 0)
+			(type default)
+		)
+	)
+	(wire
+		(pts
 			(xy 477.52 20.32) (xy 477.52 22.86)
 		)
@@
 	(wire
 		(pts
+			(xy 285.75 110.49) (xy 289.56 110.49)
+		)
+		(stroke
+			(width 0)
+			(type default)
+		)
+	)
+	(wire
+		(pts
 			(xy 392.43 38.1) (xy 392.43 48.26)
 		)
@@
 	(wire
 		(pts
-			(xy 283.21 100.33) (xy 280.67 100.33)
+			(xy 285.75 100.33) (xy 280.67 100.33)
 		)
 		(stroke
@@
 	)
 	(symbol
+		(lib_id "easyeda2kicad:AO3407A")
+		(at 360.68 227.33 90)
+		(unit 1)
+		(body_style 1)
+		(exclude_from_sim no)
+		(in_bom yes)
+		(on_board yes)
+		(in_pos_files yes)
+		(dnp no)
+		(fields_autoplaced yes)
+		(property "Reference" "Q7"
+			(at 360.68 217.17 90)
+			(show_name no)
+			(do_not_autoplace no)
+			(effects
+				(font
+					(size 1.27 1.27)
+				)
+			)
+		)
+		(property "Value" "AO3407A"
+			(at 360.68 219.71 90)
+			(show_name no)
+			(do_not_autoplace no)
+			(effects
+				(font
+					(size 1.27 1.27)
+				)
+			)
+		)
+		(property "Footprint" "easyeda2kicad:SOT-23-3_L2.9-W1.6-P1.90-LS2.8-BR"
+			(at 373.38 227.33 0)
+			(hide yes)
+			(show_name no)
+			(do_not_autoplace no)
+			(effects
+				(font
+					(size 1.27 1.27)
+				)
+			)
+		)
+		(property "Datasheet" "https://lcsc.com/product-detail/MOSFET_AOS_AO3407A_AO3407A_C15155.html"
+			(at 375.92 227.33 0)
+			(hide yes)
+			(show_name no)
+			(do_not_autoplace no)
+			(effects
+				(font
+					(size 1.27 1.27)
+				)
+			)
+		)
+		(property "Description" "AO3407A"
+			(at 360.68 227.33 0)
+			(hide yes)
+			(show_name no)
+			(do_not_autoplace no)
+			(effects
+				(font
+					(size 1.27 1.27)
+				)
+			)
+		)
+		(property "Manufacturer" "AOS"
+			(at 378.46 227.33 0)
+			(hide yes)
+			(show_name no)
+			(do_not_autoplace no)
+			(effects
+				(font
+					(size 1.27 1.27)
+				)
+			)
+		)
+		(property "MPN" "AO3407A"
+			(at 381 227.33 0)
+			(hide yes)
+			(show_name no)
+			(do_not_autoplace no)
+			(effects
+				(font
+					(size 1.27 1.27)
+				)
+			)
+		)
+		(property "LCSC Part" "C15155"
+			(at 383.54 227.33 0)
+			(hide yes)
+			(show_name no)
+			(do_not_autoplace no)
+			(effects
+				(font
+					(size 1.27 1.27)
+				)
+			)
+		)
+		(pin "3"
+		)
+		(pin "1"
+		)
+		(pin "2"
+		)
+		(instances
+			(project "LSwarm Drone PCB"
+				(path "/f914089f-8107-4513-a595-68edd26170d4"
+					(reference "Q7")
+					(unit 1)
+				)
+			)
+		)
+	)
+	(symbol
 		(lib_id "power:+3.3V")
 		(at 410.21 76.2 0)
@@
 	)
 	(symbol
-		(lib_id "Transistor_FET:AO3401A")
-		(at 360.68 227.33 90)
-		(unit 1)
-		(body_style 1)
-		(exclude_from_sim no)
-		(in_bom yes)
-		(on_board yes)
-		(in_pos_files yes)
-		(dnp no)
-		(property "Reference" "Q5"
-			(at 360.426 219.71 90)
-			(show_name no)
-			(do_not_autoplace no)
-			(effects
-				(font
-					(size 1.27 1.27)
-				)
-			)
-		)
-		(property "Value" "AO3401A"
-			(at 360.68 221.996 90)
-			(show_name no)
-			(do_not_autoplace no)
-			(effects
-				(font
-					(size 1.27 1.27)
-				)
-			)
-		)
-		(property "Footprint" "Package_TO_SOT_SMD:SOT-23"
-			(at 362.585 222.25 0)
-			(hide yes)
-			(show_name no)
-			(do_not_autoplace no)
-			(effects
-				(font
-					(size 1.27 1.27)
-					(italic yes)
-				)
-				(justify left)
-			)
-		)
-		(property "Datasheet" "http://www.aosmd.com/pdfs/datasheet/AO3401A.pdf"
-			(at 364.49 222.25 0)
-			(hide yes)
-			(show_name no)
-			(do_not_autoplace no)
-			(effects
-				(font
-					(size 1.27 1.27)
-				)
-				(justify left)
-			)
-		)
-		(property "Description" "-4.0A Id, -30V Vds, P-Channel MOSFET, SOT-23"
-			(at 360.68 227.33 0)
-			(hide yes)
-			(show_name no)
-			(do_not_autoplace no)
-			(effects
-				(font
-					(size 1.27 1.27)
-				)
-			)
-		)
-		(pin "1"
-		)
-		(pin "3"
-		)
-		(pin "2"
-		)
-		(instances
-			(project "LSwarm Drone PCB"
-				(path "/f914089f-8107-4513-a595-68edd26170d4"
-					(reference "Q5")
-					(unit 1)
-				)
-			)
-		)
-	)
-	(symbol
 		(lib_id "Device:C")
 		(at 441.96 26.67 180)
@@
 	(symbol
 		(lib_id "power:+3.3V")
-		(at 283.21 110.49 0)
+		(at 289.56 110.49 0)
 		(unit 1)
 		(body_style 1)
@@
 		(dnp no)
 		(property "Reference" "#PWR026"
-			(at 283.21 114.3 0)
+			(at 289.56 114.3 0)
 			(hide yes)
 			(show_name no)
@@
 		)
 		(property "Value" "+3.3V"
-			(at 283.21 105.918 0)
+			(at 289.56 105.918 0)
 			(show_name no)
 			(do_not_autoplace no)
@@
 		)
 		(property "Footprint" ""
-			(at 283.21 110.49 0)
+			(at 289.56 110.49 0)
 			(hide yes)
 			(show_name no)
@@
 		)
 		(property "Datasheet" ""
-			(at 283.21 110.49 0)
+			(at 289.56 110.49 0)
 			(hide yes)
 			(show_name no)
@@
 		)
 		(property "Description" "Power symbol creates a global label with name \"+3.3V\""
-			(at 283.21 110.49 0)
+			(at 289.56 110.49 0)
 			(hide yes)
 			(show_name no)

Commit message: finished pcb layout
Connections:
- net +3.3V: now also J1.1 (Pin_1)
- net GND: now also J1.2 (Pin_2)
- net RP2350_SWCLK: now also J1.3 (Pin_3)
- net RP2350_SWDIO: now also J1.4 (Pin_4)
Other:
- moved on the sheet: J1
Changed lines of the file:
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@@
 	(global_label "RP2350_SWDIO"
 		(shape input)
-		(at 38.1 167.64 180)
+		(at 29.21 167.64 0)
 		(fields_autoplaced yes)
 		(effects
@@
 				(size 1.27 1.27)
 			)
-			(justify right)
+			(justify left)
 		)
 		(property "Intersheetrefs" "${INTERSHEET_REFS}"
-			(at 20.903 167.64 0)
+			(at 46.407 167.64 0)
 			(hide yes)
 			(show_name no)
@@
 					(size 1.27 1.27)
 				)
-				(justify right)
+				(justify left)
 			)
 		)
@@
 	(global_label "RP2350_SWCLK"
 		(shape input)
-		(at 38.1 165.1 180)
+		(at 29.21 165.1 0)
 		(fields_autoplaced yes)
 		(effects
@@
 				(size 1.27 1.27)
 			)
-			(justify right)
+			(justify left)
 		)
 		(property "Intersheetrefs" "${INTERSHEET_REFS}"
-			(at 20.5402 165.1 0)
+			(at 46.7698 165.1 0)
 			(hide yes)
 			(show_name no)
@@
 					(size 1.27 1.27)
 				)
-				(justify right)
+				(justify left)
 			)
 		)
@@
 	(symbol
 		(lib_id "power:+3.3V")
-		(at 38.1 160.02 90)
+		(at 29.21 160.02 270)
 		(unit 1)
 		(body_style 1)
@@
 		(fields_autoplaced yes)
 		(property "Reference" "#PWR038"
-			(at 41.91 160.02 0)
+			(at 25.4 160.02 0)
 			(hide yes)
 			(show_name no)
@@
 		)
 		(property "Value" "+3.3V"
-			(at 34.29 160.0199 90)
+			(at 33.02 160.0199 90)
 			(show_name no)
 			(do_not_autoplace no)
@@
 		)
 		(property "Footprint" ""
-			(at 38.1 160.02 0)
+			(at 29.21 160.02 0)
 			(hide yes)
 			(show_name no)
@@
 		)
 		(property "Datasheet" ""
-			(at 38.1 160.02 0)
+			(at 29.21 160.02 0)
 			(hide yes)
 			(show_name no)
@@
 		)
 		(property "Description" "Power symbol creates a global label with name \"+3.3V\""
-			(at 38.1 160.02 0)
+			(at 29.21 160.02 0)
 			(hide yes)
 			(show_name no)
@@
 	(symbol
 		(lib_id "Connector:Conn_01x04_Pin")
-		(at 38.1 162.56 0)
+		(at 24.13 162.56 0)
 		(unit 1)
 		(body_style 1)
@@
 		(dnp no)
 		(property "Reference" "J1"
-			(at 40.386 155.194 0)
+			(at 26.416 155.194 0)
 			(show_name no)
 			(do_not_autoplace no)
@@
 		)
 		(property "Value" "Conn_01x04_Pin"
-			(at 40.64 157.734 0)
+			(at 26.67 157.734 0)
 			(show_name no)
 			(do_not_autoplace no)
@@
 		)
 		(property "Footprint" "Connector_PinHeader_2.54mm:PinHeader_1x04_P2.54mm_Vertical"
-			(at 38.1 162.56 0)
+			(at 24.13 162.56 0)
 			(hide yes)
 			(show_name no)
@@
 		)
 		(property "Datasheet" ""
-			(at 38.1 162.56 0)
+			(at 24.13 162.56 0)
 			(hide yes)
 			(show_name no)
@@
 		)
 		(property "Description" "Generic connector, single row, 01x04, script generated"
-			(at 38.1 162.56 0)
+			(at 24.13 162.56 0)
 			(hide yes)
 			(show_name no)
@@
 	(symbol
 		(lib_id "power:GND")
-		(at 38.1 162.56 270)
+		(at 29.21 162.56 90)
 		(unit 1)
 		(body_style 1)
@@
 		(fields_autoplaced yes)
 		(property "Reference" "#PWR039"
-			(at 31.75 162.56 0)
+			(at 35.56 162.56 0)
 			(hide yes)
 			(show_name no)
@@
 		)
 		(property "Value" "GND"
-			(at 34.29 162.5599 90)
+			(at 33.02 162.5599 90)
 			(show_name no)
 			(do_not_autoplace no)
@@
 		)
 		(property "Footprint" ""
-			(at 38.1 162.56 0)
+			(at 29.21 162.56 0)
 			(hide yes)
 			(show_name no)
@@
 		)
 		(property "Datasheet" ""
-			(at 38.1 162.56 0)
+			(at 29.21 162.56 0)
 			(hide yes)
 			(show_name no)
@@
 		)
 		(property "Description" "Power symbol creates a global label with name \"GND\" , ground"
-			(at 38.1 162.56 0)
+			(at 29.21 162.56 0)
 			(hide yes)
 			(show_name no)

Commit message: sync
Parts:
- renumbered U6 to ESP32, U4 to FLASH, LED2 to LED1, LED3 to LED2, LED4 to LED3, LED5 to LED4, U1 to RP2350
Changed lines of the file:
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@@
 		(in_pos_files yes)
 		(dnp no)
-		(property "Reference" "LED3"
+		(property "Reference" "LED2"
 			(at 432.562 31.242 0)
 			(show_name no)
@@
 			(project "LSwarm Drone PCB"
 				(path "/f914089f-8107-4513-a595-68edd26170d4"
-					(reference "LED3")
+					(reference "LED2")
 					(unit 1)
 				)
@@
 		(in_pos_files yes)
 		(dnp no)
-		(property "Reference" "U6"
-			(at 190.5 206.756 0)
+		(property "Reference" "ESP32"
+			(at 188.468 207.01 0)
 			(show_name no)
 			(do_not_autoplace no)
@@
 			(project "LSwarm Drone PCB"
 				(path "/f914089f-8107-4513-a595-68edd26170d4"
-					(reference "U6")
+					(reference "ESP32")
 					(unit 1)
 				)
@@
 		(in_pos_files yes)
 		(dnp no)
-		(property "Reference" "U1"
+		(property "Reference" "RP2350"
 			(at 163.4333 138.43 0)
 			(hide yes)
@@
 			(project "LSwarm Drone PCB"
 				(path "/f914089f-8107-4513-a595-68edd26170d4"
-					(reference "U1")
+					(reference "RP2350")
 					(unit 1)
 				)
@@
 		(in_pos_files yes)
 		(dnp no)
-		(property "Reference" "LED4"
+		(property "Reference" "LED3"
 			(at 457.962 31.242 0)
 			(show_name no)
@@
 			(project "LSwarm Drone PCB"
 				(path "/f914089f-8107-4513-a595-68edd26170d4"
-					(reference "LED4")
+					(reference "LED3")
 					(unit 1)
 				)
@@
 		(in_pos_files yes)
 		(dnp no)
-		(property "Reference" "U4"
+		(property "Reference" "FLASH"
 			(at 20.32 104.902 0)
 			(show_name no)
@@
 			(project "LSwarm Drone PCB"
 				(path "/f914089f-8107-4513-a595-68edd26170d4"
-					(reference "U4")
+					(reference "FLASH")
 					(unit 1)
 				)
@@
 		(in_pos_files yes)
 		(dnp no)
-		(property "Reference" "LED5"
+		(property "Reference" "LED4"
 			(at 483.362 31.242 0)
 			(show_name no)
@@
 			(project "LSwarm Drone PCB"
 				(path "/f914089f-8107-4513-a595-68edd26170d4"
-					(reference "LED5")
+					(reference "LED4")
 					(unit 1)
 				)
@@
 		(in_pos_files yes)
 		(dnp no)
-		(property "Reference" "LED2"
+		(property "Reference" "LED1"
 			(at 408.432 31.242 0)
 			(show_name no)
@@
 			(project "LSwarm Drone PCB"
 				(path "/f914089f-8107-4513-a595-68edd26170d4"
-					(reference "LED2")
+					(reference "LED1")
 					(unit 1)
 				)

Commit message: sync
Parts:
- removed U10: LSM6DSR, LSM6DSR:LGA-14L, symbol LSM6DSR:LSM6DSR
- added U1: LSM6DSRTR, easyeda2kicad:LGA-14_L3.0-W2.5-P0.50-BR, symbol easyeda2kicad:LSM6DSRTR
Connections:
- net +3.3V: now also U1.5 (VDDIO), U1.8 (VDD)
- net GND: now also U1.2 (SDX), U1.3 (SCX), U1.6 (GND), U1.7 (GND)
- net RP2350_GPIO_10: now also U1.12 (CS)
- net RP2350_GPIO_5: now also U1.4 (INT1)
- net RP2350_GPIO_6: now also U1.9 (INT2)
- net RP2350_GPIO_7: now also U1.13 (SCL)
- net RP2350_GPIO_8: now also U1.14 (SDA)
- net RP2350_GPIO_9: now also U1.1 (SDO/SA0)
- no-connect marks 30 -> 31
Other:
- moved on the sheet: C38, C39, C42, C43, C44, C45, C46, C47, C48, C66, C67, L5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

Commit message: sync
Parts:
- removed ANT2: ANT3216LL00R2400A, ANT3216LL00R2400A:ANTC3216X135N, symbol ANT3216LL00R2400A:ANT3216LL00R2400A
- removed C25: 10nF, Capacitor_SMD:C_0603_1608Metric, symbol Device:C
- removed J2: USB_C_Receptacle_USB2.0_16P, Connector_USB:USB_C_Receptacle_HRO_TYPE-C-31-M-12, symbol Connector:USB_C_Receptacle_USB2.0_16P
- removed R1, R2: 5.1k, Resistor_SMD:R_0603_1608Metric, symbol Device:R
- removed R4, R5: 27, Resistor_SMD:R_0603_1608Metric, symbol Device:R
- removed S2, S3, S5, S6: SKRPACE010, SKRPACE010:SW_SKRPACE010, symbol SKRPACE010:SKRPACE010
- removed U11: BMP581, BMP581:BMP581, symbol BMP581:BMP581
- removed U13: TPS61023DRLR, TPS61023DRLR:SOT563-ORI, symbol TPS61023DRLR:TPS61023DRLR
- removed U14: SN74LVC1T45DBVR, SN74LVC1T45DBVR:SOT95P280X145-6N, symbol SN74LVC1T45DBVR:SN74LVC1T45DBVR
- added C26: 10nF, Capacitor_SMD:C_0603_1608Metric, symbol Device:C
- added JP1: U.FL-R-SMT-1, easyeda2kicad:RF-SMD_FRF05002-JSS103M, symbol easyeda2kicad:U.FL-R-SMT-1
- added R29, R30, R31: 10k, Resistor_SMD:R_0603_1608Metric, symbol Device:R
- added R32, R33: 5.1k, Resistor_SMD:R_0603_1608Metric, symbol Device:R
- added R34, R35: 27, Resistor_SMD:R_0603_1608Metric, symbol Device:R
- added SW2, SW3, SW4, SW5: SKRPACE010, easyeda2kicad:KEY-SMD_4P-L4.2-W3.2-P2.20-LS4.6, symbol easyeda2kicad:SKRPACE010
- added U3: TPS61023DRLR, easyeda2kicad:SOT-563_L1.6-W1.2-P0.50-LS1.6-BR, symbol easyeda2kicad:TPS61023DRLR
- added U4: SN74LVC1T45DBVR, easyeda2kicad:SOT-23-6_L2.9-W1.6-P0.95-LS2.8-BR, symbol easyeda2kicad:SN74LVC1T45DBVR
- added U5: BMP581, easyeda2kicad:LGA-10_L2.0-W2.0-P0.50-TL_BMP581, symbol easyeda2kicad:BMP581
- added USB1: USB-TYPE-C-018, easyeda2kicad:USB-C_SMD-TYPE-C-31-M-12, symbol easyeda2kicad:USB-TYPE-C-018
- renumbered FLASH to FLASH1, LED1 to STATUS1
Connections:
- net +3.3V: now also C40.2, R30.1, R31.1, U4.1 (VCCA), U4.5 (DIR), U5.1 (VDDIO), U5.10 (VDD); no longer C41.1
- net +5V: now also U3.6 (VOUT), U4.6 (VCCB)
- net BATT_SW+: now also U3.2 (EN), U3.3 (VIN)
- net GND: now also C41.1, R18.1, C26.1, JP1.2 (GND), JP1.3 (GND), R29.1, R32.2, R33.1, SW3.4, SW4.4, SW5.4, U3.4 (GND), U4.2 (GND), U5.3 (VSS), U5.8 (VSS), U5.9 (VSS), USB1.A1 (GND), USB1.A12 (GND), USB1.B1 (GND), USB1.B12 (GND); no longer C40.2, R18.2
- net RP2350_GPIO_10: now also R31.2
- net RP2350_GPIO_11: now also R30.2, U5.6 (CSB)
- net RP2350_GPIO_14: now also SW4.1
- net RP2350_GPIO_15: now also SW5.1
- net RP2350_GPIO_25: now also U4.3 (A)
- net RP2350_GPIO_4: now also U5.7 (INT)
- net RP2350_GPIO_5: now also R29.2
- net RP2350_GPIO_7: now also U5.2 (SCK)
- net RP2350_GPIO_8: now also U5.4 (SDI)
- net RP2350_GPIO_9: now also U5.5 (SDO)
- net RP2350_USB_DM: now also R34.2
- net RP2350_USB_DP: now also R35.1
- net at R17.1: now also R18.2, U3.1 (FB); no longer R18.1
- net at R3.2: now also SW3.1
- net at C9.1, RP2350.26 (RUN): now also SW2.1
- net at R8.2: now also SW2.3
- net at R19.1: now also U4.4 (B)
- net at L5.1: now also U3.5 (SW)
- net at C61.1, L8.2: now also JP1.1 (SIG)
- new net: R35.2, USB1.A6 (DP1), USB1.B6 (DP2)
- new net: R32.1, USB1.A5 (CC1)
- new net: R34.1, USB1.A7 (DN1), USB1.B7 (DN2)
- new net: C26.2, USB1.0 (SH), USB1.1 (SH), USB1.2 (SH), USB1.3 (SH)
- new net: USB1.A4 (VBUS), USB1.A9 (VBUS), USB1.B4 (VBUS), USB1.B9 (VBUS)
- new net: R33.2, USB1.B5 (CC2)
Other:
- moved on the sheet: C40, C41, C42, C43, C66, C67, C68, L5, R17, R18, R19

Commit message: sync
Parts:
- L6: value L -> 24nH
Changed lines of the file:
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@@
 			)
 		)
-		(property "Value" "L"
+		(property "Value" "24nH"
 			(at 48.26 261.62 90)
 			(show_name no)

Commit message: sync
Parts:
- removed C52, C55: 12pF, Capacitor_SMD:C_0603_1608Metric, symbol Device:C
- removed C72: 220uF, Capacitor_Tantalum_SMD:CP_EIA-3528-21_Kemet-B, symbol Device:C
- removed L6: 24nH, Inductor_SMD:L_0805_2012Metric, symbol Device:L
- removed R18: 110k, Resistor_SMD:R_0603_1608Metric, symbol Device:R
- removed Y1: 12MHz, Crystal:Crystal_SMD_3225-4Pin_3.2x2.5mm, symbol Device:Crystal_GND24
- removed Y3: 40MHz, Crystal:Crystal_SMD_3225-4Pin_3.2x2.5mm, symbol Device:Crystal_GND24
- added C1: CL21A226MAQNNNE, easyeda2kicad:C0805, symbol easyeda2kicad:CL21A226MAQNNNE
- added R36: 820k, Resistor_SMD:R_0603_1608Metric, symbol Device:R
- added R37: 100k, Resistor_SMD:R_0603_1608Metric, symbol Device:R
- added X1: X322512MSB4SI, easyeda2kicad:CRYSTAL-SMD_4P-L3.2-W2.5-BL, symbol easyeda2kicad:X322512MSB4SI
- R17: value 806k -> 10k
Connections:
- net +5V: now also R36.1; no longer R17.2
- net BATT_SW+: now also C1.1
- net GND: now also C7.1, C8.1, C1.2, R37.2, X1.2 (GND), X1.4 (GND); no longer C7.2, C8.2
- net RP2350_XIN: now also C8.2, X1.1 (OSC1); no longer C8.1
- net at R17.1: now also SW1.2; no longer U3.1 (FB)
- net at R7.1: now also C7.2, X1.3 (OSC2); no longer C7.1
- net at Q7.1 (G), R28.1: now also R17.2; no longer SW1.2
- new net: R36.2, R37.1, U3.1 (FB)
Other:
- note removed: "ESP32 CRYSTAL"
- moved on the sheet: C7, C71Ceramic1, C8, Q7, R28, R7
