File: LSwarm Drone PCB/LSwarm Drone PCB.kicad_sch (KiCad schematic)
At the start: 118 parts, among them J2 Conn_01x06_Pin, J3 JST / BT2.0 Connector, J4 Conn_01x02_Pin, J5 Conn_01x02_Pin, J6 Conn_01x02_Pin, J7 Conn_01x02_Pin, J8 Conn_01x05_Pin, Q1 AO3400A, Q2 AO3400A, Q3 AO3400A, Q4 AO3400A, Q7 AO3407A, SW1 MSK12C02, SW2 SKRPACE010, SW3 SKRPACE010, U1 LSM6DSRTR, U12 AP2112K-3.3, U3 TPS61023DRLR, U4 SN74LVC1T45DBVR, U5 BMP581, U6 ESP32-C3-MINI-1U-N4, X1 X322512MSB4SI

Commit message: sync
Parts:
- removed J2: Conn_01x06_Pin, Connector_PinHeader_2.54mm:PinHeader_1x06_P2.54mm_Vertical, symbol Connector:Conn_01x06_Pin
- removed J8: Conn_01x05_Pin, Connector_PinHeader_2.54mm:PinHeader_1x05_P2.54mm_Vertical, symbol Connector:Conn_01x05_Pin
- added C56, C58, C59, C61: 100nf, Capacitor_SMD:C_0603_1608Metric, symbol Device:C
- added C69: 10uF, Capacitor_SMD:C_0603_1608Metric, symbol Device:C
- added L2: MPZ2012S601AT000, easyeda2kicad:L0805, symbol easyeda2kicad:MPZ2012S601AT000
- added R42: 10k, Resistor_SMD:R_0603_1608Metric, symbol Device:R
- added R43: 100k, Resistor_SMD:R_0603_1608Metric, symbol Device:R
- added TP34: ESP32_EN, TestPoint:TestPoint_Pad_1.0x1.0mm, symbol Connector:TestPoint
- added TP35: RP2350_RUN, TestPoint:TestPoint_Pad_1.0x1.0mm, symbol Connector:TestPoint
- added TP36: ESP32_BOOT, TestPoint:TestPoint_Pad_1.0x1.0mm, symbol Connector:TestPoint
- added TP37: RP2350_SWDIO, TestPoint:TestPoint_Pad_1.0x1.0mm, symbol Connector:TestPoint
- added TP38: ESP32_RX, TestPoint:TestPoint_Pad_1.0x1.0mm, symbol Connector:TestPoint
- added TP39: RP2350_SWCLK, TestPoint:TestPoint_Pad_1.0x1.0mm, symbol Connector:TestPoint
- added TP40: ESP32_TX, TestPoint:TestPoint_Pad_1.0x1.0mm, symbol Connector:TestPoint
- added TP41: ESP32_+3.3v, TestPoint:TestPoint_Pad_1.0x1.0mm, symbol Connector:TestPoint
- added TP42: ESP32_GND, TestPoint:TestPoint_Pad_1.0x1.0mm, symbol Connector:TestPoint
- added TP43: RP2350_GND, TestPoint:TestPoint_Pad_1.0x1.0mm, symbol Connector:TestPoint
- added TP44: RP2350_+3.3V, TestPoint:TestPoint_Pad_1.0x1.0mm, symbol Connector:TestPoint
- added U2: BU03, easyeda2kicad:WIRELM-SMD_BU03, symbol easyeda2kicad:BU03
Connections:
- net +3.3V: now also L2.2, R42.1, TP41.1, TP44.1
- net GND: now also C58.2, C59.2, C61.2, C69.2, R43.1, TP42.1, TP43.1, U2.16 (GND), U2.24 (GND), U2.8 (GND)
- net RP2350_GPIO_0: now also TP38.1
- net RP2350_GPIO_1: now also TP40.1
- net RP2350_GPIO_2: now also TP34.1
- net RP2350_GPIO_3: now also TP36.1
- net RP2350_RUN: now also TP35.1
- net RP2350_SWCLK: now also TP39.1
- net RP2350_SWDIO: now also TP37.1
- net at C55.1: now also C56.2; no longer U6.3 (3V3)
- net ESP32_VMON_ADC: now reaches U6.12 (IO0)
- net DW_WAKEUP: now reaches U6.13 (IO1)
- net DW_WAKEUP: now also U2.2 (WAKEUP)
- net DW_RST: now reaches U6.16 (IO10)
- net DW_RST: now also U2.3 (RSTN)
- net DW_MISO: now reaches U6.18 (IO4)
- net DW_MISO: now also U2.19 (MISO)
- net DW_MOSI: now reaches U6.19 (IO5)
- net DW_MOSI: now also U2.18 (MOSI)
- net DW_CLK: now reaches U6.20 (IO6)
- net DW_CLK: now also U2.20 (CLK)
- net DW_Sn: now reaches U6.21 (IO7)
- net DW_Sn: now also R42.2, U2.17 (CSN)
- net DW_IRQ: now reaches U6.6 (IO3)
- net DW_IRQ: now also R43.2, U2.22 (IRQ)
- new net: C56.1, U6.3 (3V3)
- new net UW_3.3V: C58.1, C59.1, C61.1, C69.1, L2.1, U2.5 (VDD), U2.6 (VCC), U2.7 (VCC)
- no-connect marks 44 -> 47
Other:
- note added: "UWB ANCHOR"
- moved on the sheet: C1, C52, C55, C71Ceramic1, Q7, R17, R18, R28, R32, SW1

Commit message: sync
Connections:
- net RP2350_GPIO_10: now also U1.13 (SCL), U5.2 (SCK); no longer R31.2, U1.12 (CS)
- net RP2350_GPIO_11: now also U1.14 (SDA), U5.4 (SDI); no longer R30.2, U5.6 (CSB)
- net RP2350_GPIO_7: now also R31.2, U1.12 (CS); no longer U1.13 (SCL), U5.2 (SCK)
- net RP2350_GPIO_8: now also U1.1 (SDO/SA0), U5.5 (SDO); no longer U1.14 (SDA), U5.4 (SDI)
- net RP2350_GPIO_9: now also R30.2, U5.6 (CSB); no longer U1.1 (SDO/SA0), U5.5 (SDO)
