File: LSwarm Drone PCB/LSwarm Drone PCB.kicad_pcb (KiCad board)
At the start: 4 copper layers, 100 x 99.8 mm, 142 parts, among them J2 Conn_01x06_Pin, J3 JST / BT2.0 Connector, J4 Conn_01x02_Pin, J5 Conn_01x02_Pin, J6 Conn_01x02_Pin, J7 Conn_01x02_Pin, J8 Conn_01x05_Pin, Q1 AO3400A, Q2 AO3400A, Q3 AO3400A, Q4 AO3400A, Q7 AO3407A, SW1 MSK12C02, SW2 SKRPACE010, SW3 SKRPACE010, U1 LSM6DSRTR, U12 AP2112K-3.3, U3 TPS61023DRLR, U4 SN74LVC1T45DBVR, U5 BMP581, U6 ESP32-C3-MINI-1U-N4, X1 X322512MSB4SI

Commit message: sync
Parts:
- removed J2: Conn_01x06_Pin, Connector_PinHeader_2.54mm:PinHeader_1x06_P2.54mm_Vertical
- removed J8: Conn_01x05_Pin, Connector_PinHeader_2.54mm:PinHeader_1x05_P2.54mm_Vertical
- added C56: 100nf, Capacitor_SMD:C_0603_1608Metric, F.Cu at (23.2, 58.0)
- added C58: 100nf, Capacitor_SMD:C_0603_1608Metric, B.Cu at (29.7, 42.0)
- added C59: 100nf, Capacitor_SMD:C_0603_1608Metric, B.Cu at (28.2, 42.0)
- added C61: 100nf, Capacitor_SMD:C_0603_1608Metric, B.Cu at (26.7, 42.0)
- added C69: 10uF, Capacitor_SMD:C_0603_1608Metric, B.Cu at (25.2, 42.0)
- added L2: MPZ2012S601AT000, easyeda2kicad:L0805, B.Cu at (23.2, 41.5)
- added R42: 10k, Resistor_SMD:R_0603_1608Metric, B.Cu at (30.0, 60.8)
- added R43: 100k, Resistor_SMD:R_0603_1608Metric, B.Cu at (21.9, 60.2)
- added TP34: ESP32_EN, TestPoint:TestPoint_Pad_1.0x1.0mm, F.Cu at (71.5, 31.5)
- added TP35: RP2350_RUN, TestPoint:TestPoint_Pad_1.0x1.0mm, F.Cu at (39.8, 69.2)
- added TP36: ESP32_BOOT, TestPoint:TestPoint_Pad_1.0x1.0mm, F.Cu at (69.5, 31.5)
- added TP37: RP2350_SWDIO, TestPoint:TestPoint_Pad_1.0x1.0mm, F.Cu at (37.8, 69.2)
- added TP38: ESP32_RX, TestPoint:TestPoint_Pad_1.0x1.0mm, F.Cu at (75.5, 31.5)
- added TP39: RP2350_SWCLK, TestPoint:TestPoint_Pad_1.0x1.0mm, F.Cu at (35.8, 69.2)
- added TP40: ESP32_TX, TestPoint:TestPoint_Pad_1.0x1.0mm, F.Cu at (73.5, 31.5)
- added TP41: ESP32_+3.3v, TestPoint:TestPoint_Pad_1.0x1.0mm, F.Cu at (67.5, 31.5)
- added TP42: ESP32_GND, TestPoint:TestPoint_Pad_1.0x1.0mm, F.Cu at (65.5, 31.5)
- added TP43: RP2350_GND, TestPoint:TestPoint_Pad_1.0x1.0mm, F.Cu at (33.8, 69.2)
- added TP44: RP2350_+3.3V, TestPoint:TestPoint_Pad_1.0x1.0mm, F.Cu at (31.8, 69.2)
- added U2: BU03, easyeda2kicad:WIRELM-SMD_BU03, B.Cu at (26.3, 51.5)
- moved dino 4.59 mm to (72.2, 34.8)
- moved dino 3.75 mm to (68.5, 52.6)
- moved dino 3.03 mm to (59.0, 37.5)
- moved C55 0.55 mm to (23.2, 59.5), turned to 0 degrees
Connections:
- C55 pad 1: Net-(U6-3V3) -> Net-(C55-Pad1)
- U6 pad 12: unconnected-(U6-IO0-Pad12) -> ESP32_VMON_ADC
- U6 pad 13: unconnected-(U6-IO1-Pad13) -> DW_WAKEUP
- U6 pad 16: unconnected-(U6-IO10-Pad16) -> DW_RST
- U6 pad 18: unconnected-(U6-IO4-Pad18) -> DW_MISO
- U6 pad 19: unconnected-(U6-IO5-Pad19) -> DW_MOSI
- U6 pad 20: unconnected-(U6-IO6-Pad20) -> DW_CLK
- U6 pad 21: unconnected-(U6-IO7-Pad21) -> DW_Sn
- U6 pad 6: unconnected-(U6-IO3-Pad6) -> DW_IRQ
Routing:
- net DW_WAKEUP: track 0.00 -> 41.0 mm, vias 0 -> 3
- net DW_RST: track 0.00 -> 36.2 mm, vias 0 -> 1
- net +5V: track 318.5 -> 300.6 mm
- net UW_3.3V: track 0.00 -> 17.0 mm
- net GND: track 192.1 -> 207.8 mm, vias 113 -> 119
- net DW_Sn: track 0.00 -> 13.2 mm, vias 0 -> 1
- net DW_CLK: track 0.00 -> 12.9 mm, vias 0 -> 1
- net RP2350_GPIO_25_5.5V: track 98.2 -> 87.4 mm
- net DW_MOSI: track 0.00 -> 10.8 mm, vias 0 -> 1
- net DW_MISO: track 0.00 -> 10.4 mm, vias 0 -> 1
- net DW_IRQ: track 0.00 -> 8.27 mm, vias 0 -> 1
- net RP2350_GPIO_1: track 94.2 -> 89.7 mm
- net RP2350_SWCLK: track 34.2 -> 31.3 mm
- net RP2350_GPIO_0: track 94.3 -> 91.9 mm
- net RP2350_SWDIO: track 33.1 -> 30.9 mm
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